File: DS1722_Temp_Sensor/_autosave-DS1722_Temp_Sensor.kicad_sch (KiCad schematic)
At the start: 13 parts, among them J1 Conn_01x08, J2 Conn_01x08

Commit message: Working on Layout, but I'm about to crash. Need sleep. Turning in incomplete :(
Connections:
- net PICO: no longer J1.6 (Pin_6)
- net POCI: now also J1.6 (Pin_6)
Changed lines of the file:
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@@
 		)
 	)
-	(label "PICO"
+	(label "POCI"
 		(at 78.74 67.31 0)
 		(fields_autoplaced yes)
